Commit message: Updates Ouster LiDAR mesh and position
Updates the Ouster LiDAR mesh to use the correct visual model.

Adjusts the position of the LDR12 LiDAR in the robot configuration
for better placement.

File: husarion_components_description/urdf/ouster.urdf.xacro (robot description, xacro)
@@ -65,12 +65,12 @@
     </joint>
     <link name="${prefix}ouster_${model}_link">
-      <!-- <visual>
+      <visual>
         <origin xyz="0.0 0.0 0.0" rpy="0.0 0.0 0.0" />
         <geometry>
-          <mesh filename="package://husarion_components_description/meshes/${mesh}.dae" />
+          <mesh filename="package://husarion_components_description/meshes/ouster_lidar.dae" />
         </geometry>
-      </visual> -->
+      </visual>
       <!-- TODO Remove simple visuals when mesh is ready -->
-      <visual>
+      <!-- <visual>
         <origin xyz="0.0 0.0 0.0" rpy="0.0 0.0 0.0" />
         <geometry>
@@ -80,5 +80,5 @@
           <color rgba="0.6 0.6 0.6 1.0" />
         </material>
-      </visual>
+      </visual> -->
       <collision>
         <origin xyz="0.0 0.0 ${0.072/2.0}" rpy="0.0 0.0 0.0" />

Commit message: Adds inertial parameters to Ouster lidar link
Adds inertial parameters to the Ouster lidar link in the URDF.
This is required for proper simulation, as the link previously had no inertial properties defined.

File: husarion_components_description/urdf/ouster.urdf.xacro (robot description, xacro)
@@ -100,5 +100,13 @@
       <child link="${prefix}os_lidar" />
     </joint>
-    <link name="${prefix}os_lidar" />
+    <link name="${prefix}os_lidar">
+      <inertial>
+        <origin xyz="0.0 0.0 0.0" rpy="0.0 0.0 0.0" />
+        <mass value="0.001" />
+        <inertia ixx="1e-6" ixy="0.0" ixz="0.0"
+                           iyy="1e-6" iyz="0.0"
+                                      izz="1e-6" />
+      </inertial>
+    </link>
     <gazebo reference="${prefix}os_lidar">
       <!-- gpu_lidar has to be set, CPU lidar doesn't work in ignition -
